File: PCB/Final-Year_v1.0/final_year v1.0.kicad_pcb (KiCad board)
At the start: 2 copper layers, 147.3 x 104.1 mm, 45 parts, among them J1 Power In, J2 Screw_Terminal_01x07, J3 Screw_Terminal_01x03, J4 Screw_Terminal_01x04, J5 Screw_Terminal_01x03, J6 PT1000, J7 HCPV 22x, J8 LDR_module, J9 Screw_Terminal_01x03, Q1 2N3904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

Commit message: address to gnd and decoupling cap to ads
Parts:
- added C9: 0.1uF, Capacitor_THT:C_Disc_D6.0mm_W2.5mm_P5.00mm, F.Cu at (149.9, 61.0)
- BZ1: footprint Buzzer:Buzzer_12x9.5RM7.6 -> Buzzer_Beeper:Buzzer_12x9.5RM7.6
Connections:
- U6 pad 6: unconnected-(U6-ADDR-Pad6) -> GND
Changed lines of the file:
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@@
   (net 48 "LDR")
   (net 49 "unconnected-(U6-ALRT-Pad5)")
-  (net 50 "unconnected-(U6-ADDR-Pad6)")
   (footprint "LED_THT:LED_D5.0mm_IRGrey" (layer "F.Cu")
     (at 72.38 99.065)
@@
   )
   (footprint "Capacitor_THT:C_Disc_D6.0mm_W2.5mm_P5.00mm" (layer "F.Cu")
+    (at 149.94 60.96)
+    (descr "C, Disc series, Radial, pin pitch=5.00mm, , diameter*width=6*2.5mm^2, Capacitor, http://cdn-reichelt.de/documents/datenblatt/B300/DS_KERKO_TC.pdf")
+    (tags "C Disc series Radial pin pitch 5.00mm  diameter 6mm width 2.5mm Capacitor")
+    (property "Sheetfile" "final_year v1.0.kicad_sch")
+    (property "Sheetname" "")
+    (property "ki_description" "Unpolarized capacitor")
+    (property "ki_keywords" "cap capacitor")
+    (attr through_hole)
+    (fp_text reference "C9" (at 2.5 -2.5) (layer "F.SilkS")
+        (effects (font (size 1 1) (thickness 0.15)))
+    )
+    (fp_text value "0.1uF" (at 2.5 2.5) (layer "F.Fab")
+        (effects (font (size 1 1) (thickness 0.15)))
+    )
+    (fp_text user "${REFERENCE}" (at 2.5 0) (layer "F.Fab")
+        (effects (font (size 1 1) (thickness 0.15)))
+    )
+    (fp_line (start -0.62 -1.37) (end -0.62 -0.925)
+      (stroke (width 0.12) (type solid)) (layer "F.SilkS"))
+    (fp_line (start -0.62 -1.37) (end 5.62 -1.37)
+      (stroke (width 0.12) (type solid)) (layer "F.SilkS"))
+    (fp_line (start -0.62 0.925) (end -0.62 1.37)
+      (stroke (width 0.12) (type solid)) (layer "F.SilkS"))
+    (fp_line (start -0.62 1.37) (end 5.62 1.37)
+      (stroke (width 0.12) (type solid)) (layer "F.SilkS"))
+    (fp_line (start 5.62 -1.37) (end 5.62 -0.925)
+      (stroke (width 0.12) (type solid)) (layer "F.SilkS"))
+    (fp_line (start 5.62 0.925) (end 5.62 1.37)
+      (stroke (width 0.12) (type solid)) (layer "F.SilkS"))
+    (fp_line (start -1.05 -1.5) (end -1.05 1.5)
+      (stroke (width 0.05) (type solid)) (layer "F.CrtYd"))
+    (fp_line (start -1.05 1.5) (end 6.05 1.5)
+      (stroke (width 0.05) (type solid)) (layer "F.CrtYd"))
+    (fp_line (start 6.05 -1.5) (end -1.05 -1.5)
+      (stroke (width 0.05) (type solid)) (layer "F.CrtYd"))
+    (fp_line (start 6.05 1.5) (end 6.05 -1.5)
+      (stroke (width 0.05) (type solid)) (layer "F.CrtYd"))
+    (fp_line (start -0.5 -1.25) (end -0.5 1.25)
+      (stroke (width 0.1) (type solid)) (layer "F.Fab"))
+    (fp_line (start -0.5 1.25) (end 5.5 1.25)
+      (stroke (width 0.1) (type solid)) (layer "F.Fab"))
+    (fp_line (start 5.5 -1.25) (end -0.5 -1.25)
+      (stroke (width 0.1) (type solid)) (layer "F.Fab"))
+    (fp_line (start 5.5 1.25) (end 5.5 -1.25)
+      (stroke (width 0.1) (type solid)) (layer "F.Fab"))
+    (pad "1" thru_hole circle (at 0 0) (size 1.6 1.6) (drill 0.8) (layers "*.Cu" "*.Mask")
+      (net 3 "GND") (pintype "passive"))
+    (pad "2" thru_hole circle (at 5 0) (size 1.6 1.6) (drill 0.8) (layers "*.Cu" "*.Mask")
+      (net 4 "+5V") (pintype "passive"))
+    (model "${KICAD6_3DMODEL_DIR}/Capacitor_THT.3dshapes/C_Disc_D6.0mm_W2.5mm_P5.00mm.wrl"
+      (offset (xyz 0 0 0))
+      (scale (xyz 1 1 1))
+      (rotate (xyz 0 0 0))
+    )
+  )
+  (footprint "Capacitor_THT:C_Disc_D6.0mm_W2.5mm_P5.00mm" (layer "F.Cu")
     (at 149.94 47.23)
     (descr "C, Disc series, Radial, pin pitch=5.00mm, , diameter*width=6*2.5mm^2, Capacitor, http://cdn-reichelt.de/documents/datenblatt/B300/DS_KERKO_TC.pdf")
@@
       (net 49 "unconnected-(U6-ALRT-Pad5)") (pinfunction "ALRT") (pintype "output+no_connect"))
     (pad "6" thru_hole circle (at -1.27 6.6675) (size 1.508 1.508) (drill 1) (layers "*.Cu" "*.Mask")
-      (net 50 "unconnected-(U6-ADDR-Pad6)") (pinfunction "ADDR") (pintype "input+no_connect"))
+      (net 3 "GND") (pinfunction "ADDR") (pintype "input"))
     (pad "7" thru_hole circle (at -3.81 6.6675) (size 1.508 1.508) (drill 1) (layers "*.Cu" "*.Mask")
       (net 26 "SDA") (pinfunction "SDA") (pintype "bidirectional"))
@@
     )
   )
-  (footprint "Buzzer:Buzzer_12x9.5RM7.6" (layer "F.Cu")
+  (footprint "Buzzer_Beeper:Buzzer_12x9.5RM7.6" (layer "F.Cu")
     (at 107.46 99.06)
     (descr "Generic Buzzer, D12mm height 9.5mm with RM7.6mm")
@@
     (pad "2" thru_hole circle (at 7.6 0) (size 2 2) (drill 1) (layers "*.Cu" "*.Mask")
       (net 2 "Net-(BZ1-+)") (pinfunction "+") (pintype "passive"))
-    (model "${KISYS3DMOD}/Buzzer_Beeper.3dshapes/Buzzer_12x9.5RM7.6.wrl"
-      (offset (xyz 0 0 0))
-      (scale (xyz 1 1 1))
+    (model "${KICAD6_3DMODEL_DIR}/Buzzer_Beeper.3dshapes/Buzzer_12x9.5RM7.6.wrl"
+      (offset (xyz 0 0 0))
+      (scale (xyz 1 1 1))
