File: PCB/Final-Year_v1.0/final_year v1.0.kicad_pcb (KiCad board)
At the start: 2 copper layers, 37 parts, among them J1 Power In, J2 Screw_Terminal_01x07, J3 Screw_Terminal_01x03, J4 Screw_Terminal_01x04, J5 Screw_Terminal_01x03, J6 PT1000, J7 HCPV 22x, J8 LDR, J9 Screw_Terminal_01x03, U1 LM7805_TO220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

Commit message: Add files via upload
Parts:
- added BZ1: Buzzer, Buzzer_Beeper:Buzzer_15x7.5RM7.6, F.Cu at (91.4, 104.6)
- added C1: 0.1u, Capacitor_THT:C_Disc_D6.0mm_W2.5mm_P5.00mm, F.Cu at (68.6, 57.8)
- added C7: 10nF, Capacitor_THT:C_Disc_D3.8mm_W2.6mm_P2.50mm, F.Cu at (20.3, 32.4)
- added C8: 0.1uF, Capacitor_THT:C_Disc_D6.0mm_W2.5mm_P5.00mm, F.Cu at (74.9, 33.1)
- added D1: LED, LED_THT:LED_D5.0mm, F.Cu at (74.1, 106.1)
- added Q1: BC547, Package_TO_SOT_THT:TO-92_Inline, F.Cu at (61.8, 83.3)
- added R19: 1.2k, Resistor_THT:R_Axial_DIN0207_L6.3mm_D2.5mm_P10.16mm_Horizontal, F.Cu at (57.1, 83.8)
- added R20: 330, Resistor_THT:R_Axial_DIN0207_L6.3mm_D2.5mm_P10.16mm_Horizontal, F.Cu at (47.6, 88.3)
- C2: footprint Capacitor_THT:C_Radial_D6.3mm_H7.0mm_P2.50mm -> Capacitor_THT:CP_Radial_D4.0mm_P2.00mm
- C3: footprint Capacitor_THT:C_Radial_D6.3mm_H5.0mm_P2.50mm -> Capacitor_THT:CP_Radial_D4.0mm_P2.00mm
- J5: value Screw_Terminal_01x03 -> Actuator
- moved J3 37.7 mm to (26.6, 105.1)
- moved J4 35.9 mm to (46.9, 105.1)
- moved R17 15.2 mm to (50.5, 60.3)
- moved R16 15.2 mm to (63.5, 60.3)
- moved R3 10.9 mm to (26.1, 48.0), turned to -90 degrees
- moved R2 10.8 mm to (22.3, 58.1), turned to 90 degrees
- moved C6 8.56 mm to (41.9, 39.9)
- moved C4 8.07 mm to (60.3, 35.6)
- moved C2 7.25 mm to (55.1, 36.1)
- moved U2 6.83 mm to (66.7, 38.6)
- moved R1 6.83 mm to (54.4, 31.2)
- moved U1 6.83 mm to (49.6, 38.1)
- moved R18 6.36 mm to (43.2, 84.5)
- moved C3 5.94 mm to (37.5, 39.7)
- moved C5 4.38 mm to (29.2, 88.9)
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Connections:
- J2 pad 1: TX0 -> D13
- J2 pad 2: RX0 -> D14
- J2 pad 3: D18 -> TX0
- J2 pad 4: D15 -> RX0
- J2 pad 5: D14 -> D18
- J2 pad 6: D13 -> D15
- U4 pad 22: unconnected-(U4-D33-Pad22) -> D33
- U4 pad 27: unconnected-(U4-D12-Pad27) -> D12
- U6 pad 1: LDR -> Battery_level
- U6 pad 2: Battery_level -> PT1000
- U6 pad 3: HCPV -> LDR
- U6 pad 4: PT1000 -> HCPV
- U6 pad 6: unconnected-(U6-ADDR-Pad6) -> GND
Routing:
- net +5V: track 0.00 -> 255.2 mm
- net +12V: track 0.00 -> 250.2 mm
- net TX0: track 0.00 -> 66.5 mm
- net RX0: track 0.00 -> 65.5 mm
- net D18: track 0.00 -> 59.4 mm
- net D4: track 0.00 -> 56.4 mm, vias 0 -> 2
- net D5: track 0.00 -> 55.7 mm
- net Net-(U5B-+): track 0.00 -> 51.1 mm, vias 0 -> 1
- net D14: track 0.00 -> 48.1 mm
- net D15: track 0.00 -> 45.4 mm
- net PT1000: track 0.00 -> 44.9 mm
- net Net-(J6-Pin_1): track 0.00 -> 41.7 mm
- net D13: track 0.00 -> 40.9 mm
- net LDR: track 0.00 -> 40.2 mm
- net D2: track 0.00 -> 40.0 mm
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- added copper zone on B.Cu, net GND
Other:
- board outline added: 90 x 100 mm

Commit message: Add files via upload
Parts:
- added H1: MountingHole, MountingHole:MountingHole_3.2mm_M3, F.Cu at (80.8, 29.1)
- added H2: MountingHole, MountingHole:MountingHole_3.2mm_M3, F.Cu at (77.2, 96.2)
- added H3: MountingHole, MountingHole:MountingHole_3.2mm_M3, F.Cu at (18.8, 30.5)
- added H4: MountingHole, MountingHole:MountingHole_3.2mm_M3, F.Cu at (18.8, 100.2)
- moved C7 4.75 mm to (25.1, 32.1)
- moved R8 2.55 mm to (28.6, 32.2)
- moved R7 2.55 mm to (28.6, 28.7)
Routing:
- net D2: track 40.0 -> 115.9 mm
- net Net-(J4-Pin_2): track 24.3 -> 69.6 mm
- net +12V: track 250.2 -> 261.9 mm
- net Net-(U5B-+): track 51.1 -> 46.5 mm
- net GND: track 9.58 -> 6.50 mm, vias 1 -> 0
- net D4: track 56.4 -> 58.1 mm
- net D15: track 45.4 -> 47.1 mm
- net Net-(J6-Pin_1): track 41.7 -> 43.2 mm
- added copper zone on F.Cu, net GND
Other:
- board text added: "+"
- board text added: "+12"
- board text added: "+5"
- board text added: "+5V"
- board text added: "-"
- board text added: "AOut"
- board text added: "D13"
- board text added: "D14"
- board text added: "D15"
- board text added: "D18"
- board text added: "D2"
- board text added: "D32"
- board text added: "D34"
- board text added: "D4"
- board text added: "D5"
- board text added: "Dust Sensor"
- board text added: "GND"
- board text added: "HCPV-22x"
- board text added: "LDR"
- board text added: "MQ2"
- board text added: "Motor"
- board text added: "PT1000"
- board text added: "Power In"
- board text added: "Rx0"
- board text added: "Tx0"

Commit message: gerber files added
Parts:
- moved Q1 2.85 mm to (62.9, 80.6)
Routing:
- net Net-(Q1-B): track 4.96 -> 6.50 mm
Changed lines of the file:
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@@
       (plot_on_all_layers_selection 0x0000000_00000000)
       (disableapertmacros false)
-      (usegerberextensions false)
-      (usegerberattributes true)
-      (usegerberadvancedattributes true)
-      (creategerberjobfile true)
+      (usegerberextensions true)
+      (usegerberattributes false)
+      (usegerberadvancedattributes false)
+      (creategerberjobfile false)
       (dashed_line_dash_ratio 12.000000)
       (dashed_line_gap_ratio 3.000000)
@@
       (plotinvisibletext false)
       (sketchpadsonfab false)
-      (subtractmaskfromsilk false)
+      (subtractmaskfromsilk true)
       (outputformat 1)
       (mirror false)
-      (drillshape 1)
+      (drillshape 0)
       (scaleselection 1)
-      (outputdirectory "")
+      (outputdirectory "Gerber/")
     )
   )
@@
   )
   (footprint "Package_TO_SOT_THT:TO-92_Inline" (layer "F.Cu")
-    (at 61.805 83.295 -90)
+    (at 62.865 80.645 -90)
     (descr "TO-92 leads in-line, narrow, oval pads, drill 0.75mm (see NXP sot054_po.pdf)")
     (tags "to-92 sc-43 sc-43a sot54 PA33 transistor")
@@
   (segment (start 68.62 57.785) (end 62.357 57.785) (width 0.254) (layer "F.Cu") (net 26))
   (segment (start 56.007 60.325) (end 60.452 55.88) (width 0.254) (layer "F.Cu") (net 26))
-  (segment (start 61.805 83.295) (end 77.695 83.295) (width 0.254) (layer "F.Cu") (net 32))
-  (segment (start 77.695 83.295) (end 91.365 96.965) (width 0.254) (layer "F.Cu") (net 32))
+  (segment (start 75.045 80.645) (end 62.865 80.645) (width 0.254) (layer "F.Cu") (net 32))
+  (segment (start 91.365 96.965) (end 75.045 80.645) (width 0.254) (layer "F.Cu") (net 32))
   (segment (start 71.525 102.005) (end 71.525 106.065) (width 0.254) (layer "F.Cu") (net 36))
   (segment (start 57.785 88.265) (end 71.525 102.005) (width 0.254) (layer "F.Cu") (net 36))
@@
   (segment (start 79.629 60.325) (end 63.5 60.325) (width 0.254) (layer "F.Cu") (net 46))
   (segment (start 92.456 47.498) (end 79.629 60.325) (width 0.254) (layer "F.Cu") (net 46))
-  (segment (start 57.15 83.82) (end 57.895 84.565) (width 0.254) (layer "F.Cu") (net 47))
-  (segment (start 57.895 84.565) (end 61.805 84.565) (width 0.254) (layer "F.Cu") (net 47))
+  (segment (start 59.055 81.915) (end 62.865 81.915) (width 0.254) (layer "F.Cu") (net 47))
+  (segment (start 57.15 83.82) (end 59.055 81.915) (width 0.254) (layer "F.Cu") (net 47))
   (segment (start 39.645 85.285) (end 39.645 92.71) (width 0.254) (layer "F.Cu") (net 48))
   (segment (start 43.265 81.665) (end 39.645 85.285) (width 0.254) (layer "F.Cu") (net 48))
